File: First.kicad_pcb (KiCad board)
At the start: 4 copper layers, 53 parts, among them J1 Conn_01x04_Female, J2 Conn_01x04_Female, J3 USB_B_Micro, J4 Conn_01x04_Female, J5 Conn_01x04_Female, J6 Conn_01x04_Female, J7 Conn_01x04_Female, J8 Conn_01x04_Female, J9 Conn_01x04_Female, U1 CP2102N-A01-GQFN24, U2 TUSB2046IBVFR, U3 LM1117IMP-3.3_NOPB, U4 CP2102N-A01-GQFN24, U5 CP2102N-A01-GQFN24, U6 CP2102N-A01-GQFN24, Y1 FQ7050B-7.3728

Commit message: Totally new version
Parts:
- removed C14, C15, C16: 22p, Capacitor_SMD:C_0603_1608Metric
- removed C17: 100u, Capacitor_SMD:C_0603_1608Metric
- removed J6, J8: Conn_01x04_Female, Connector_PinSocket_2.54mm:PinSocket_1x04_P2.54mm_Vertical
- removed J7, J9: Conn_01x04_Female, Connector_JST:JST_EH_B4B-EH-A_1x04_P2.50mm_Vertical
- added D1: LED, LED_THT:LED_D3.0mm, F.Cu at (134.3, 65.1)
- added JP1: 48MCLK_JMP, Jumper:SolderJumper-2_P1.3mm_Bridged_RoundedPad1.0x1.5mm, F.Cu at (126.1, 45.3)
- added R20: 470, Resistor_SMD:R_0603_1608Metric, F.Cu at (137.9, 65.0)
- C1: value 100u -> 22p
- C10, C11: value 27u -> 22p
- C12: value 100u -> 20p
- C13: value 22p -> 20p
- C2: value 1u -> 10u
- C6: value 0.1u -> 22p
- C9: value 100u -> 10u
- J1: value Conn_01x04_Female -> UART0; footprint Connector_JST:JST_EH_B4B-EH-A_1x04_P2.50mm_Vertical -> Connector_PinSocket_2.54mm:PinSocket_1x05_P2.54mm_Vertical
- J2: value Conn_01x04_Female -> UART1; footprint Connector_PinSocket_2.54mm:PinSocket_1x04_P2.54mm_Vertical -> Connector_PinSocket_2.54mm:PinSocket_1x05_P2.54mm_Vertical
- J4: value Conn_01x04_Female -> UART2; footprint Connector_JST:JST_EH_B4B-EH-A_1x04_P2.50mm_Vertical -> Connector_PinSocket_2.54mm:PinSocket_1x05_P2.54mm_Vertical
- J5: value Conn_01x04_Female -> UART3; footprint Connector_PinSocket_2.54mm:PinSocket_1x04_P2.54mm_Vertical -> Connector_PinSocket_2.54mm:PinSocket_1x05_P2.54mm_Vertical
- R10, R11, R17, R19: value 15k -> 27
- R12, R16, R8, R9: value 27 -> 15k
- U1: value CP2102N-A01-GQFN24 -> CP2102N-DEV0
- U2: footprint TUSB2046IBVFR:TUSB2046IBVFR -> TUSB2046:TUSB2046IBVFR
- U3: value LM1117IMP-3.3_NOPB -> CP2102N-DEV1; footprint LM1117:LM1117IMP-3.3&slash_NOPB -> Package_DFN_QFN:QFN-24-1EP_4x4mm_P0.5mm_EP2.6x2.6mm
- U4: value CP2102N-A01-GQFN24 -> CP2102N_DEV2
- U5: value CP2102N-A01-GQFN24 -> LD1086V33-DG; footprint Package_DFN_QFN:QFN-24-1EP_4x4mm_P0.5mm_EP2.6x2.6mm -> Package_TO_SOT_THT:TO-220-3_Vertical
- Y1: value FQ7050B-7.3728 -> HC49SDLF-8.00MHz; footprint FQ7050:OSC_FQ7050B-7.3728 -> HC49:HC49SDLF800MHz
- moved C2 90.8 mm to (103.0, 51.5), turned to -90 degrees
- moved C12 80.8 mm to (114.2, 42.6), turned to 0 degrees
- moved C9 76.9 mm to (104.5, 51.5), turned to -90 degrees
- moved C13 75.4 mm to (117.2, 42.6), turned to 180 degrees
- moved U5 74.4 mm to (104.2, 46.2), turned to 180 degrees
- moved C6 68.5 mm to (124.7, 60.3)
- moved R17 64.4 mm to (124.3, 53.3), turned to -135 degrees
- moved R19 64.1 mm to (123.2, 52.2), turned to -135 degrees
- moved U6 62.4 mm to (132.0, 50.4)
- moved C8 61.4 mm to (124.7, 55.7), turned to 0 degrees
- moved J5 60.2 mm to (140.4, 41.1), turned to -90 degrees
- moved J2 60.1 mm to (145.0, 70.0)
- moved J3 59.8 mm to (99.0, 54.5)
- moved R10 59.5 mm to (120.7, 64.9), turned to 135 degrees
- moved R15 59.4 mm to (124.7, 57.2)
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Connections:
- C1 pad 1: VDD -> /D-1
- C10 pad 1: GND -> /D-3
- C10 pad 2: Net-(C10-Pad2) -> GND
- C11 pad 1: Net-(C11-Pad1) -> /D+3
- C12 pad 1: VDD -> Net-(C12-Pad1)
- C13 pad 1: /2_D- -> Net-(C13-Pad1)
- C3 pad 1: /4_D- -> /D-0
- C5 pad 1: /4_D+ -> /D+0
- C6 pad 1: VBUS -> /D-2
- C7 pad 1: /1_D- -> /D+1
- C8 pad 1: /1_D+ -> /D+2
- C9 pad 1: VDD -> +3V3
- J1 pad 1: Net-(J1-Pad1) -> GND
- J1 pad 2: Net-(J1-Pad2) -> /CTS_0
- J1 pad 3: Net-(J1-Pad3) -> /RTS_0
- J1 pad 4: Net-(J1-Pad4) -> /RX_0
- J2 pad 1: Net-(J1-Pad1) -> GND
- J2 pad 2: Net-(J1-Pad2) -> /CTS_1
- J2 pad 3: Net-(J1-Pad3) -> /RTS_1
- J2 pad 4: Net-(J1-Pad4) -> /RX_1
- J3 pad 2: /USB_D- -> /USB_IN-
- J3 pad 3: /USB_D+ -> /USB_IN+
- J3 pad 4: Net-(J3-Pad4) -> unconnected-(J3-Pad4)
- J4 pad 1: Net-(J4-Pad1) -> GND
- J4 pad 2: Net-(J4-Pad2) -> /CTS_2
- J4 pad 3: Net-(J4-Pad3) -> /RTS_2
- J4 pad 4: Net-(J4-Pad4) -> /RX_2
- J5 pad 1: Net-(J5-Pad1) -> GND
- J5 pad 2: Net-(J5-Pad2) -> /CTS_3
- J5 pad 3: Net-(J5-Pad3) -> /RTS_3
- J5 pad 4: Net-(J5-Pad4) -> /RX_3
- R1 pad 2: /4_D- -> /U0_OUT-
- R10 pad 1: GND -> /U1_OUT-
- R10 pad 2: /1_D+ -> /D-1
- R11 pad 1: GND -> /U2_OUT-
- R11 pad 2: /1_D- -> /D-2
- R12 pad 1: /3_D+ -> GND
- R12 pad 2: /3_D+ -> /U1_OUT+
- R13 pad 2: /3_D+ -> /U2_OUT+
- R14 pad 1: /2_D+ -> /U1_OUT+
- R14 pad 2: /2_D+ -> /D+1
- R15 pad 1: /2_D- -> /U2_OUT+
- R15 pad 2: /2_D- -> /D+2
- R16 pad 1: /3_D- -> GND
- R16 pad 2: /3_D- -> /U3_OUT-
- R17 pad 1: GND -> /U3_OUT-
- R17 pad 2: /2_D- -> /D-3
- R18 pad 2: /3_D- -> /U3_OUT+
- R19 pad 1: GND -> /U3_OUT+
- R19 pad 2: /2_D+ -> /D+3
- R2 pad 1: /4_D- -> /U0_OUT-
- R2 pad 2: /4_D- -> /D-0
- R3 pad 2: /4_D+ -> /U0_OUT+
- R4 pad 1: /4_D+ -> /U0_OUT+
- R4 pad 2: /4_D+ -> /D+0
- R5 pad 1: /USB_D- -> /USB_D+
- R5 pad 2: /USB_D- -> /USB_IN+
- R6 pad 1: /USB_D+ -> /USB_IN-
- R6 pad 2: /USB_D+ -> /USB_D-
- R7 pad 1: VDD -> +3V3
- R8 pad 1: /1_D+ -> GND
- R8 pad 2: /1_D+ -> /U1_OUT-
- R9 pad 1: /1_D- -> GND
- R9 pad 2: /1_D- -> /U2_OUT-
- U1 pad 1: Net-(U1-Pad1) -> unconnected-(U1-Pad1)
- U1 pad 10: Net-(U1-Pad10) -> unconnected-(U1-Pad10)
- U1 pad 11: Net-(U1-Pad11) -> unconnected-(U1-Pad11)
- U1 pad 12: Net-(U1-Pad12) -> unconnected-(U1-Pad12)
- U1 pad 13: Net-(U1-Pad13) -> unconnected-(U1-Pad13)
- U1 pad 14: Net-(U1-Pad14) -> unconnected-(U1-Pad14)
- U1 pad 15: Net-(U1-Pad15) -> unconnected-(U1-Pad15)
- U1 pad 16: Net-(U1-Pad16) -> unconnected-(U1-Pad16)
- U1 pad 17: Net-(U1-Pad17) -> unconnected-(U1-Pad17)
- U1 pad 18: Net-(J4-Pad1) -> /CTS_0
- U1 pad 19: Net-(J4-Pad2) -> /RTS_0
- U1 pad 2: Net-(U1-Pad2) -> GND
- U1 pad 20: Net-(J4-Pad3) -> /RX_0
- U1 pad 21: Net-(J4-Pad4) -> /TX_0
- U1 pad 22: Net-(U1-Pad22) -> unconnected-(U1-Pad22)
- U1 pad 23: Net-(U1-Pad23) -> unconnected-(U1-Pad23)
- U1 pad 24: Net-(U1-Pad24) -> unconnected-(U1-Pad24)
- U1 pad 3: /4_D+ -> /U0_OUT+
- U1 pad 4: /4_D- -> /U0_OUT-
- U1 pad 5: Net-(U1-Pad5) -> unconnected-(U1-Pad5)
- U1 pad 6: VDD -> unconnected-(U1-Pad6)
- U1 pad 9: Net-(U1-Pad9) -> unconnected-(U1-Pad9)
- U2 pad 10: Net-(U2-Pad10) -> unconnected-(U2-Pad10)
- U2 pad 11: /4_D- -> /D-0
- U2 pad 12: /4_D+ -> /D+0
- U2 pad 13: Net-(U2-Pad13) -> unconnected-(U2-Pad13)
- U2 pad 14: Net-(U2-Pad14) -> unconnected-(U2-Pad14)
- U2 pad 15: /1_D- -> /D-1
- U2 pad 16: /1_D+ -> /D+1
- U2 pad 17: Net-(U2-Pad17) -> unconnected-(U2-Pad17)
- U2 pad 18: Net-(U2-Pad18) -> unconnected-(U2-Pad18)
- U2 pad 19: /2_D- -> /D-2
- U2 pad 20: /2_D+ -> /D+2
- U2 pad 21: Net-(U2-Pad21) -> unconnected-(U2-Pad21)
- U2 pad 22: Net-(U2-Pad22) -> unconnected-(U2-Pad22)
- U2 pad 23: /3_D- -> /D-3
- U2 pad 24: /3_D+ -> /D+3
- U2 pad 25: VDD -> +3V3
- U2 pad 26: VDD -> +3V3
- U2 pad 27: Net-(U2-Pad27) -> Net-(JP1-Pad1)
- U2 pad 28: Net-(U2-Pad27) -> GND
- U2 pad 29: Net-(C10-Pad2) -> Net-(C13-Pad1)
- U2 pad 3: Net-(U2-Pad3) -> +3V3
- U2 pad 30: Net-(C11-Pad1) -> Net-(C12-Pad1)
- U2 pad 31: Net-(U2-Pad31) -> unconnected-(U2-Pad31)
- U2 pad 32: Net-(U2-Pad32) -> /STATUS_LED
- U2 pad 4: Net-(U2-Pad4) -> unconnected-(U2-Pad4)
- U2 pad 5: Net-(U2-Pad5) -> unconnected-(U2-Pad5)
- U2 pad 6: GND -> unconnected-(U2-Pad6)
- U2 pad 9: Net-(U2-Pad9) -> unconnected-(U2-Pad9)
- U3 pad 1: GND -> unconnected-(U3-Pad1)
- U3 pad 2: Net-(U3-Pad2) -> GND
- U3 pad 3: VBUS -> /U1_OUT+
- U3 pad 4: VDD -> /U1_OUT-
- U4 pad 1: Net-(U4-Pad1) -> unconnected-(U4-Pad1)
- U4 pad 10: Net-(U4-Pad10) -> unconnected-(U4-Pad10)
- U4 pad 11: Net-(U4-Pad11) -> unconnected-(U4-Pad11)
- U4 pad 12: Net-(U4-Pad12) -> unconnected-(U4-Pad12)
- U4 pad 13: Net-(U4-Pad13) -> unconnected-(U4-Pad13)
- U4 pad 14: Net-(U4-Pad14) -> unconnected-(U4-Pad14)
- U4 pad 15: Net-(U4-Pad15) -> unconnected-(U4-Pad15)
- U4 pad 16: Net-(U4-Pad16) -> unconnected-(U4-Pad16)
- U4 pad 17: Net-(U4-Pad17) -> unconnected-(U4-Pad17)
- U4 pad 18: Net-(J1-Pad1) -> /CTS_2
- U4 pad 19: Net-(J1-Pad2) -> /RTS_2
- U4 pad 20: Net-(J1-Pad3) -> /RX_2
- U4 pad 21: Net-(J1-Pad4) -> /TX_2
- U4 pad 22: Net-(U4-Pad22) -> unconnected-(U4-Pad22)
- U4 pad 23: Net-(U4-Pad23) -> unconnected-(U4-Pad23)
- U4 pad 24: Net-(U4-Pad24) -> unconnected-(U4-Pad24)
- U4 pad 25: Net-(U4-Pad25) -> GND
- U4 pad 3: /1_D+ -> /U2_OUT+
- U4 pad 4: /1_D- -> /U2_OUT-
- U4 pad 5: Net-(U4-Pad5) -> unconnected-(U4-Pad5)
- U4 pad 6: VDD -> unconnected-(U4-Pad6)
- U4 pad 9: Net-(U4-Pad9) -> unconnected-(U4-Pad9)
- U5 pad 1: Net-(U5-Pad1) -> GND
- U5 pad 2: Net-(U5-Pad2) -> +3V3
- U5 pad 3: /3_D+ -> VBUS
- U6 pad 1: Net-(U6-Pad1) -> unconnected-(U6-Pad1)
- U6 pad 10: Net-(U6-Pad10) -> unconnected-(U6-Pad10)
- U6 pad 11: Net-(U6-Pad11) -> unconnected-(U6-Pad11)
- U6 pad 12: Net-(U6-Pad12) -> unconnected-(U6-Pad12)
- U6 pad 13: Net-(U6-Pad13) -> unconnected-(U6-Pad13)
- U6 pad 14: Net-(U6-Pad14) -> unconnected-(U6-Pad14)
- U6 pad 15: Net-(U6-Pad15) -> unconnected-(U6-Pad15)
- U6 pad 16: Net-(U6-Pad16) -> unconnected-(U6-Pad16)
- U6 pad 17: Net-(U6-Pad17) -> unconnected-(U6-Pad17)
- U6 pad 18: Net-(J8-Pad1) -> /CTS_3
- U6 pad 19: Net-(J8-Pad2) -> /RTS_3
- U6 pad 2: Net-(U6-Pad2) -> GND
- U6 pad 20: Net-(J8-Pad3) -> /RX_3
- U6 pad 21: Net-(J8-Pad4) -> /TX_3
- U6 pad 22: Net-(U6-Pad22) -> unconnected-(U6-Pad22)
- U6 pad 23: Net-(U6-Pad23) -> unconnected-(U6-Pad23)
- U6 pad 24: Net-(U6-Pad24) -> unconnected-(U6-Pad24)
- U6 pad 3: /2_D+ -> /U3_OUT+
- U6 pad 4: /2_D- -> /U3_OUT-
- U6 pad 5: Net-(U6-Pad5) -> unconnected-(U6-Pad5)
- U6 pad 6: VDD -> unconnected-(U6-Pad6)
- U6 pad 9: Net-(U6-Pad9) -> unconnected-(U6-Pad9)
- Y1 pad 1: Net-(C10-Pad2) -> Net-(C12-Pad1)
- Y1 pad 2: (no net) -> Net-(C13-Pad1)
Routing:
- net +3V3: track 0.00 -> 34.5 mm, vias 0 -> 4
- net /CTS_0: track 0.00 -> 32.2 mm
- net /RTS_0: track 0.00 -> 30.8 mm
- net /RX_0: track 0.00 -> 29.5 mm
- net /TX_0: track 0.00 -> 28.6 mm
- net Net-(J5-Pad3): track 27.4 -> 0.00 mm, vias 1 -> 0
- net /STATUS_LED: track 0.00 -> 27.2 mm
- net Net-(J5-Pad4): track 26.7 -> 0.00 mm, vias 1 -> 0
- net Net-(J5-Pad2): track 25.9 -> 0.00 mm, vias 1 -> 0
- net VDD: track 25.5 -> 0.00 mm, vias 9 -> 0
- net Net-(J5-Pad1): track 24.3 -> 0.00 mm, vias 1 -> 0
- net /TX_1: track 0.00 -> 21.8 mm
- net Net-(J1-Pad1): track 21.7 -> 0.00 mm, vias 1 -> 0
- net Net-(J1-Pad2): track 21.1 -> 0.00 mm, vias 1 -> 0
- net Net-(J1-Pad4): track 20.0 -> 0.00 mm, vias 1 -> 0
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- added copper zone on B.Cu, net GND
- added copper zone on F.Cu, net GND
- removed copper zone on GND.Cu, net GND
- removed copper zone on F.Cu, net VDD
- removed copper zone on VDD.Cu, net VDD
Other:
- board outline added: 54.1 x 51.8 mm
- copper layers 4 -> 2
- net class Default removed

Commit message: Ordered version
Parts:
- added C14: 22p, Capacitor_SMD:C_0603_1608Metric, B.Cu at (132.2, 61.3)
- added C15: 22p, Capacitor_SMD:C_0603_1608Metric, B.Cu at (122.6, 73.6)
- added C16: 22p, Capacitor_SMD:C_0603_1608Metric, B.Cu at (133.0, 53.6)
- added C17: 22p, Capacitor_SMD:C_0603_1608Metric, B.Cu at (112.0, 71.7)
- added G***: LOGO, LOGO, B.Cu at (116.0, 63.8)
- added R21: 10k, Resistor_SMD:R_0603_1608Metric, F.Cu at (114.8, 74.7)
- added R22: 10k, Resistor_SMD:R_0603_1608Metric, F.Cu at (133.6, 70.4)
- added R23: 10k, Resistor_SMD:R_0603_1608Metric, F.Cu at (134.8, 57.4)
- added R24: 10k, Resistor_SMD:R_0603_1608Metric, F.Cu at (136.5, 47.7)
- D1: footprint LED_THT:LED_D3.0mm -> LED_SMD:LED_0805_2012Metric
- moved J1 11.8 mm to (141.0, 73.9), turned to -90 degrees
- moved J3 1.38 mm to (97.6, 54.5)
- moved D1 1.09 mm to (133.2, 65.1)
- moved J5 0.63 mm to (141.0, 41.1)
- moved C12 0.20 mm to (114.2, 42.4)
- moved C13 0.20 mm to (117.2, 42.4)
- moved Y1 0.20 mm to (115.5, 46.7)
Connections:
- U1 pad 15: unconnected-(U1-Pad15) -> Net-(U1-Pad15)
- U3 pad 15: unconnected-(U3-Pad15) -> Net-(U3-Pad15)
- U4 pad 15: unconnected-(U4-Pad15) -> Net-(U4-Pad15)
- U6 pad 15: unconnected-(U6-Pad15) -> Net-(U6-Pad15)
Routing:
- net /TX_0: track 28.6 -> 14.6 mm
- net /RX_0: track 29.5 -> 17.4 mm
- net /RTS_0: track 30.8 -> 20.1 mm
- net /CTS_0: track 32.2 -> 23.8 mm
- net VBUS: track 77.5 -> 84.2 mm
- net GND: track 22.2 -> 28.6 mm, vias 83 -> 78
- net Net-(U3-Pad15): track 0.00 -> 5.31 mm
- net Net-(U6-Pad15): track 0.00 -> 3.53 mm
- net Net-(U4-Pad15): track 0.00 -> 1.73 mm
- net Net-(U1-Pad15): track 0.00 -> 1.66 mm
- net /D-2: track 3.22 -> 4.76 mm
- net /D+2: track 3.22 -> 4.76 mm
- net /USB_IN+: track 7.50 -> 8.86 mm
- net /USB_IN-: track 7.50 -> 8.86 mm
- net /CTS_3: track 12.5 -> 13.1 mm
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Other:
- board size 54.1 x 51.8 mm -> 55.6 x 41.1 mm
- board text added: "CT"
- board text added: "GND"
- board text added: "RT"
- board text added: "RX"
- board text added: "TX"

Commit message: Final and tested version
Parts:
- removed JP1: 48MCLK_JMP, Jumper:SolderJumper-2_P1.3mm_Bridged_RoundedPad1.0x1.5mm
- added D2: LED, LED_SMD:LED_0805_2012Metric, F.Cu at (107.2, 65.5)
- added H1: MountingHole_Pad, MountingHole:MountingHole_2.2mm_M2_Pad_Via, F.Cu at (146.5, 40.7)
- added H2: MountingHole_Pad, MountingHole:MountingHole_2.2mm_M2_Pad_Via, F.Cu at (98.5, 40.9)
- added H3: MountingHole_Pad, MountingHole:MountingHole_2.2mm_M2_Pad_Via, F.Cu at (98.6, 74.5)
- added H4: MountingHole_Pad, MountingHole:MountingHole_2.2mm_M2_Pad_Via, F.Cu at (146.6, 74.6)
- added R25: 470, Resistor_SMD:R_0603_1608Metric, F.Cu at (107.2, 61.8)
- Y1: value HC49SDLF-8.00MHz -> HC49SDLF-6.00MHz
- moved R20 32.9 mm to (105.2, 61.8), turned to 90 degrees
- moved D1 28.0 mm to (105.2, 65.6), turned to 90 degrees
Connections:
- D1 pad 1: Net-(D1-Pad1) -> GND
- D1 pad 2: /STATUS_LED -> Net-(D1-Pad2)
- R20 pad 1: GND -> Net-(D1-Pad2)
- R20 pad 2: Net-(D1-Pad1) -> VBUS
- U2 pad 10: unconnected-(U2-Pad10) -> +3V3
- U2 pad 14: unconnected-(U2-Pad14) -> +3V3
- U2 pad 18: unconnected-(U2-Pad18) -> +3V3
- U2 pad 22: unconnected-(U2-Pad22) -> +3V3
- U2 pad 27: Net-(JP1-Pad1) -> GND
- U2 pad 31: unconnected-(U2-Pad31) -> GND
- U2 pad 32: /STATUS_LED -> unconnected-(U2-Pad32)
- U2 pad 4: unconnected-(U2-Pad4) -> +3V3
- U2 pad 6: unconnected-(U2-Pad6) -> GND
Routing:
- net /STATUS_LED: track 27.7 -> 0.00 mm
- net +3V3: track 34.5 -> 60.7 mm
- net Net-(JP1-Pad1): track 12.8 -> 0.00 mm
- net Net-(D1-Pad1): track 2.95 -> 0.00 mm
- net Net-(D1-Pad2): track 0.00 -> 1.98 mm
- net GND: track 28.6 -> 30.6 mm, vias 78 -> 80
- net Net-(D2-Pad2): track 0.00 -> 1.96 mm
- net VBUS: track 84.2 -> 86.2 mm, vias 4 -> 5
Other:
- board text added: "3v3"
- board text added: "5V0"

Commit message: Second review
Parts:
- removed H1, H2, H3, H4: MountingHole_Pad, MountingHole:MountingHole_2.2mm_M2_Pad_Via
- added 5V_ON: SolderJumper_2_Bridged, Jumper:SolderJumper-2_P1.3mm_Bridged_RoundedPad1.0x1.5mm, B.Cu at (124.3, 40.4)
- added C19: 22p, Capacitor_SMD:C_0603_1608Metric, B.Cu at (131.4, 63.1)
- added C20: 22p, Capacitor_SMD:C_0603_1608Metric, B.Cu at (123.3, 73.8)
- added C21: 4.7u, Capacitor_SMD:C_0603_1608Metric, B.Cu at (113.8, 67.7)
- added C22: 22p, Capacitor_SMD:C_0603_1608Metric, B.Cu at (129.2, 49.9)
- added D10: LED, LED_SMD:LED_0805_2012Metric, F.Cu at (141.8, 52.4)
- added D3: LED, LED_SMD:LED_0805_2012Metric, F.Cu at (136.5, 61.0)
- added D4: LED, LED_SMD:LED_0805_2012Metric, F.Cu at (112.0, 76.3)
- added D5: LED, LED_SMD:LED_0805_2012Metric, F.Cu at (129.1, 75.0)
- added D6: LED, LED_SMD:LED_0805_2012Metric, F.Cu at (136.5, 58.9)
- added D7: LED, LED_SMD:LED_0805_2012Metric, F.Cu at (114.0, 76.3)
- added D8: LED, LED_SMD:LED_0805_2012Metric, F.Cu at (130.5, 73.6)
- added D9: LED, LED_SMD:LED_0805_2012Metric, F.Cu at (139.9, 52.4)
- added JP1: SolderJumper_2_Bridged, Jumper:SolderJumper-2_P1.3mm_Bridged_RoundedPad1.0x1.5mm, B.Cu at (125.1, 80.0)
- added JP2: SolderJumper_2_Bridged, Jumper:SolderJumper-2_P1.3mm_Bridged_RoundedPad1.0x1.5mm, B.Cu at (146.8, 62.8)
- added JP3: SolderJumper_2_Bridged, Jumper:SolderJumper-2_P1.3mm_Bridged_RoundedPad1.0x1.5mm, B.Cu at (145.2, 39.7)
- added R26: 1k, Resistor_SMD:R_0603_1608Metric, F.Cu at (133.3, 61.5)
- added R27: 1k, Resistor_SMD:R_0603_1608Metric, F.Cu at (112.0, 68.2)
- added R28: 1k, Resistor_SMD:R_0603_1608Metric, B.Cu at (125.4, 70.7)
- added R29: 10k, Resistor_SMD:R_0603_1608Metric, F.Cu at (135.1, 56.4)
- added R30: 10k, Resistor_SMD:R_0603_1608Metric, F.Cu at (131.6, 71.2)
- added R31: 300, Resistor_SMD:R_0603_1608Metric, B.Cu at (139.5, 55.6)
- added R32: 1k, Resistor_SMD:R_0603_1608Metric, B.Cu at (131.3, 52.1)
- added R33: 10k, Resistor_SMD:R_0603_1608Metric, F.Cu at (136.0, 47.5)
- C14: value 22p -> 4.7u; moved to F.Cu
- C15, C16: value 22p -> 4.7u
- J1, J2, J4, J5: footprint Connector_PinSocket_2.54mm:PinSocket_1x05_P2.54mm_Vertical -> Connector_PinSocket_2.54mm:PinSocket_1x06_P2.54mm_Vertical
- R22: value 10k -> 300
- R23, R24: value 10k -> 300; moved to B.Cu
- U1: footprint Package_DFN_QFN:QFN-24-1EP_4x4mm_P0.5mm_EP2.6x2.6mm -> CP2102:QFN50P400X400X80-25N
- U3: value CP2102N-DEV1 -> CP2102N-DEV0; footprint Package_DFN_QFN:QFN-24-1EP_4x4mm_P0.5mm_EP2.6x2.6mm -> CP2102:QFN50P400X400X80-25N
- U4: value CP2102N_DEV2 -> CP2102N-DEV0; footprint Package_DFN_QFN:QFN-24-1EP_4x4mm_P0.5mm_EP2.6x2.6mm -> CP2102:QFN50P400X400X80-25N
- U5: value LD1086V33-DG -> LM1117-3.3; footprint Package_TO_SOT_THT:TO-220-3_Vertical -> Package_TO_SOT_SMD:SOT-223; moved to B.Cu
- U6: value CP2102N-A01-GQFN24 -> CP2102N-DEV0; footprint Package_DFN_QFN:QFN-24-1EP_4x4mm_P0.5mm_EP2.6x2.6mm -> CP2102:QFN50P400X400X80-25N
- moved R23 23.2 mm to (115.3, 70.1), turned to 90 degrees
- moved C15 20.7 mm to (132.3, 55.4)
- moved R24 20.1 mm to (127.8, 65.9), turned to 180 degrees
- moved C16 16.6 mm to (125.1, 68.3), turned to 135 degrees
- moved J1 14.3 mm to (128.2, 80.2), turned to 90 degrees
- moved R22 13.8 mm to (137.4, 57.1)
- moved J4 12.9 mm to (146.8, 42.2), turned to 0 degrees
- moved U4 12.9 mm to (127.1, 70.2), turned to -45 degrees
- moved U3 12.8 mm to (131.2, 58.0), turned to 0 degrees
- moved J5 12.8 mm to (128.2, 40.4), turned to 90 degrees
- moved J2 4.47 mm to (146.8, 65.9), turned to 0 degrees
- moved G*** 4.01 mm to (116.5, 59.8)
- moved C17 3.72 mm to (111.3, 68.0), turned to 180 degrees
- moved U5 2.87 mm to (101.5, 45.1), turned to 90 degrees
- moved C14 2.01 mm to (133.3, 63.0)
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Connections:
- C14 pad 1: VBUS -> +3V3
- C15 pad 1: VBUS -> +3V3
- C16 pad 1: VBUS -> +3V3
- J1 pad 1: GND -> Net-(J1-Pad1)
- J1 pad 2: /CTS_0 -> /TX_0
- J1 pad 3: /RTS_0 -> /RX_0
- J1 pad 4: /RX_0 -> /RTS_0
- J1 pad 5: /TX_0 -> /CTS_0
- J2 pad 1: GND -> Net-(J2-Pad1)
- J2 pad 2: /CTS_1 -> /TX_1
- J2 pad 3: /RTS_1 -> /RX_1
- J2 pad 4: /RX_1 -> /RTS_1
- J2 pad 5: /TX_1 -> /CTS_1
- J4 pad 1: GND -> Net-(J4-Pad1)
- J4 pad 2: /CTS_2 -> /TX_2
- J4 pad 3: /RTS_2 -> /RX_2
- J4 pad 4: /RX_2 -> /RTS_2
- J4 pad 5: /TX_2 -> /CTS_2
- J5 pad 1: GND -> Net-(J5-Pad1)
- J5 pad 2: /CTS_3 -> /TX_3
- J5 pad 3: /RTS_3 -> /RX_3
- J5 pad 4: /RX_3 -> /RTS_3
- J5 pad 5: /TX_3 -> /CTS_3
- R22 pad 1: GND -> Net-(D3-Pad2)
- R22 pad 2: Net-(R22-Pad2) -> +3V3
- R23 pad 1: GND -> Net-(D4-Pad2)
- R23 pad 2: Net-(R23-Pad2) -> +3V3
- R24 pad 1: GND -> Net-(D5-Pad2)
- R24 pad 2: Net-(R24-Pad2) -> +3V3
- U1 pad 13: unconnected-(U1-Pad13) -> Net-(D4-Pad1)
- U1 pad 14: unconnected-(U1-Pad14) -> Net-(D7-Pad1)
- U1 pad 5: unconnected-(U1-Pad5) -> +3V3
- U1 pad 6: unconnected-(U1-Pad6) -> +3V3
- U1 pad 7: VBUS -> +3V3
- U1 pad 9: unconnected-(U1-Pad9) -> Net-(R27-Pad1)
- U3 pad 13: unconnected-(U3-Pad13) -> Net-(D3-Pad1)
- U3 pad 14: unconnected-(U3-Pad14) -> Net-(D6-Pad1)
- U3 pad 15: Net-(R22-Pad2) -> Net-(R29-Pad2)
- U3 pad 18: /CTS_1 -> /CTS_2
- U3 pad 19: /RTS_1 -> /RTS_2
- U3 pad 20: /RX_1 -> /RX_2
- U3 pad 21: /TX_1 -> /TX_2
- U3 pad 3: /U1_OUT+ -> /U2_OUT+
- U3 pad 4: /U1_OUT- -> /U2_OUT-
- U3 pad 5: unconnected-(U3-Pad5) -> +3V3
- U3 pad 6: unconnected-(U3-Pad6) -> +3V3
- U3 pad 7: VBUS -> +3V3
- U3 pad 9: unconnected-(U3-Pad9) -> Net-(R26-Pad1)
- U4 pad 13: unconnected-(U4-Pad13) -> Net-(D5-Pad1)
- U4 pad 14: unconnected-(U4-Pad14) -> Net-(D8-Pad1)
- U4 pad 15: Net-(R23-Pad2) -> Net-(R30-Pad2)
- U4 pad 18: /CTS_2 -> /CTS_1
- U4 pad 19: /RTS_2 -> /RTS_1
- U4 pad 20: /RX_2 -> /RX_1
- U4 pad 21: /TX_2 -> /TX_1
- U4 pad 3: /U2_OUT+ -> /U1_OUT+
- U4 pad 4: /U2_OUT- -> /U1_OUT-
- U4 pad 5: unconnected-(U4-Pad5) -> +3V3
- U4 pad 6: unconnected-(U4-Pad6) -> +3V3
- U4 pad 7: VBUS -> +3V3
- U4 pad 9: unconnected-(U4-Pad9) -> Net-(R28-Pad1)
- U6 pad 13: unconnected-(U6-Pad13) -> Net-(D9-Pad1)
- U6 pad 14: unconnected-(U6-Pad14) -> Net-(D10-Pad1)
- U6 pad 15: Net-(R24-Pad2) -> Net-(R33-Pad2)
- U6 pad 5: unconnected-(U6-Pad5) -> +3V3
- U6 pad 6: unconnected-(U6-Pad6) -> +3V3
- U6 pad 7: VBUS -> +3V3
- U6 pad 9: unconnected-(U6-Pad9) -> Net-(R32-Pad1)
Routing:
- net VBUS: track 86.2 -> 289.6 mm, vias 5 -> 6
- net +3V3: track 60.7 -> 140.6 mm, vias 4 -> 12
- net Net-(D5-Pad2): track 0.00 -> 14.8 mm, vias 0 -> 1
- net Net-(D10-Pad1): track 0.00 -> 10.5 mm, vias 0 -> 2
- net Net-(D4-Pad2): track 0.00 -> 9.06 mm, vias 0 -> 1
- net /RTS_0: track 20.1 -> 28.8 mm, vias 0 -> 2
- net /CTS_0: track 23.8 -> 32.3 mm, vias 0 -> 2
- net Net-(D9-Pad1): track 0.00 -> 7.91 mm, vias 0 -> 2
- net /RX_0: track 17.4 -> 25.2 mm, vias 0 -> 2
- net /TX_0: track 14.6 -> 22.3 mm, vias 0 -> 2
- net Net-(D10-Pad2): track 0.00 -> 6.47 mm, vias 0 -> 1
- net Net-(R22-Pad2): track 5.31 -> 0.00 mm
- net Net-(R27-Pad1): track 0.00 -> 5.15 mm
- net Net-(R26-Pad1): track 0.00 -> 4.13 mm
- net Net-(D3-Pad2): track 0.00 -> 4.13 mm
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Other:
- board size 55.6 x 41.1 mm -> 55.6 x 46.9 mm
- board text added: "*"
- board text added: "5V"
- board text added: "R T"
- board text added: "Radosław Sajdak"
- board text added: "UART-USB HUB"
- board text added: "UART0"
- board text added: "UART1"
- board text added: "UART2"
- board text added: "UART3"
- board text added: "github.com/RadoslawSajdak"
