File: First.kicad_sch (KiCad schematic)
At the start: 48 parts, among them J1 UART0, J2 UART1, J3 USB_B_Micro, J4 UART2, J5 UART3, U1 CP2102N-DEV0, U2 TUSB2046IBVFR, U3 CP2102N-DEV1, U4 CP2102N_DEV2, U5 LD1086V33-DG, U6 CP2102N-A01-GQFN24, Y1 HC49SDLF-8.00MHz

Commit message: Ordered version
Parts:
- added C14, C15, C16, C17: 22p, Capacitor_SMD:C_0603_1608Metric, symbol First-rescue:CP-Device
- added R21, R22, R23, R24: 10k, Resistor_SMD:R_0603_1608Metric, symbol Device:R
- D1: footprint LED_THT:LED_D3.0mm -> LED_SMD:LED_0805_2012Metric
Connections:
- net GND: now also C14.2, C15.2, C16.2, C17.2, R21.1, R22.1, R23.1, R24.1
- net VBUS: now also C14.1, C15.1, C16.1, C17.1
- net at U1.15 (~{SUSPENDb}): now also R21.2
- net at U3.15 (~{SUSPENDb}): now also R22.2
- net at U6.15 (~{SUSPENDb}): now also R24.2
- net at U4.15 (~{SUSPENDb}): now also R23.2
- no-connect marks 65 -> 61

Commit message: Final and tested version
Parts:
- removed JP1: 48MCLK_JMP, Jumper:SolderJumper-2_P1.3mm_Bridged_RoundedPad1.0x1.5mm, symbol Jumper:SolderJumper_2_Bridged
- added D2: LED, LED_SMD:LED_0805_2012Metric, symbol Device:LED
- added H1, H2, H3, H4: MountingHole_Pad, MountingHole:MountingHole_2.2mm_M2_Pad_Via, symbol Mechanical:MountingHole_Pad
- added R25: 470, Resistor_SMD:R_0603_1608Metric, symbol Device:R
- Y1: value HC49SDLF-8.00MHz -> HC49SDLF-6.00MHz
Connections:
- net +3V3: now also U2.10 (*OVRCUR1), U2.14 (*OVRCUR2), U2.18 (*OVRCUR3), U2.22 (*OVRCUR4), U2.4 (*RESET), R25.2
- net GND: now also D1.1 (K), U2.27 (TSTPLL/48MCLK), U2.31 (TSTMODE), U2.6 (EEDATA/GANGED), D2.1 (K), H1.1, H2.1, H3.1, H4.1; no longer R20.1
- net VBUS: now also R20.2
- net STATUS_LED: no longer names the net of U2.32 (SUSPEND)
- net STATUS_LED: no longer D1.2 (A)
- new net: D1.2 (A), R20.1
- new net: D2.2 (A), R25.1
- no-connect marks 61 -> 55
Other:
- company: (none) -> Radosław Sajdak
- title: (none) -> UART-USB converters HUB
- moved on the sheet: C12, C13, Y1

Commit message: Second review
Parts:
- removed C14, C15, C16, C17: 22p, Capacitor_SMD:C_0603_1608Metric, symbol First-rescue:CP-Device
- removed H1, H2, H3, H4: MountingHole_Pad, MountingHole:MountingHole_2.2mm_M2_Pad_Via, symbol Mechanical:MountingHole_Pad
- removed J1: UART0, Connector_PinSocket_2.54mm:PinSocket_1x05_P2.54mm_Vertical, symbol Connector:Conn_01x05_Male
- removed J2: UART1, Connector_PinSocket_2.54mm:PinSocket_1x05_P2.54mm_Vertical, symbol Connector:Conn_01x05_Male
- removed J4: UART2, Connector_PinSocket_2.54mm:PinSocket_1x05_P2.54mm_Vertical, symbol Connector:Conn_01x05_Male
- removed J5: UART3, Connector_PinSocket_2.54mm:PinSocket_1x05_P2.54mm_Vertical, symbol Connector:Conn_01x05_Male
- removed U5: LD1086V33-DG, Package_TO_SOT_THT:TO-220-3_Vertical, symbol Regulator_Linear:LD1086V33-DG
- added C14, C15, C16, C21: 4.7u, Capacitor_SMD:C_0603_1608Metric, symbol Device:C
- added C17, C19, C20, C22: 22p, Capacitor_SMD:C_0603_1608Metric, symbol Device:C
- added D10, D3, D4, D5, D6, D7, D8, D9: LED, LED_SMD:LED_0805_2012Metric, symbol Device:LED
- added J1: UART0, Connector_PinSocket_2.54mm:PinSocket_1x06_P2.54mm_Vertical, symbol Connector:Conn_01x06_Female
- added J2: UART1, Connector_PinSocket_2.54mm:PinSocket_1x06_P2.54mm_Vertical, symbol Connector:Conn_01x06_Female
- added J4: UART2, Connector_PinSocket_2.54mm:PinSocket_1x06_P2.54mm_Vertical, symbol Connector:Conn_01x06_Female
- added J5: UART3, Connector_PinSocket_2.54mm:PinSocket_1x06_P2.54mm_Vertical, symbol Connector:Conn_01x06_Female
- added JP1, JP2, JP3, JP4: SolderJumper_2_Bridged, Jumper:SolderJumper-2_P1.3mm_Bridged_RoundedPad1.0x1.5mm, symbol Jumper:SolderJumper_2_Bridged
- added R26, R27, R28, R32: 1k, Resistor_SMD:R_0603_1608Metric, symbol Device:R
- added R29, R30, R33: 10k, Resistor_SMD:R_0603_1608Metric, symbol Device:R
- added R31: 300, Resistor_SMD:R_0603_1608Metric, symbol Device:R
- added U5: LM1117-3.3, Package_TO_SOT_SMD:SOT-223, symbol Regulator_Linear:LM1117-3.3
- R22, R23, R24: value 10k -> 300
- U1: footprint Package_DFN_QFN:QFN-24-1EP_4x4mm_P0.5mm_EP2.6x2.6mm -> CP2102:QFN50P400X400X80-25N
- U3: value CP2102N-DEV1 -> CP2102N-DEV0; footprint Package_DFN_QFN:QFN-24-1EP_4x4mm_P0.5mm_EP2.6x2.6mm -> CP2102:QFN50P400X400X80-25N
- U4: value CP2102N_DEV2 -> CP2102N-DEV0; footprint Package_DFN_QFN:QFN-24-1EP_4x4mm_P0.5mm_EP2.6x2.6mm -> CP2102:QFN50P400X400X80-25N
- U6: value CP2102N-A01-GQFN24 -> CP2102N-DEV0; footprint Package_DFN_QFN:QFN-24-1EP_4x4mm_P0.5mm_EP2.6x2.6mm -> CP2102:QFN50P400X400X80-25N
Connections:
- net +3V3: now also R22.2, R23.2, R24.2, U1.5 (VIO), U1.6 (VDD), U1.7 (REGIN), U3.5 (VIO), U3.6 (VDD), U3.7 (REGIN), U4.5 (VIO), U4.6 (VDD), U4.7 (REGIN), U6.5 (VIO), U6.6 (VDD), U6.7 (REGIN), C14.1, C15.1, C16.1, C21.1, R26.2, R27.2, R28.2, R31.2, R32.2, U5.2 (VO)
- net CTS_0: now also J1.5 (Pin_5)
- net CTS_1: now also U4.18 (CTS), J2.5 (Pin_5); no longer U3.18 (CTS)
- net CTS_2: now also U3.18 (CTS), J4.5 (Pin_5); no longer U4.18 (CTS)
- net CTS_3: now also J5.5 (Pin_5)
- net GND: now also C14.2, C15.2, C16.2, C17.2, C19.2, C20.2, C21.2, C22.2, J1.6 (Pin_6), J2.6 (Pin_6), J4.6 (Pin_6), J5.6 (Pin_6), R29.1, R30.1, R33.1, U5.1 (GND); no longer R22.1, R23.1, R24.1
- net RTS_0: now also J1.4 (Pin_4)
- net RTS_1: now also U4.19 (RTS), J2.4 (Pin_4); no longer U3.19 (RTS)
- net RTS_2: now also U3.19 (RTS), J4.4 (Pin_4); no longer U4.19 (RTS)
- net RTS_3: now also J5.4 (Pin_4)
- net RX_0: now also J1.3 (Pin_3)
- net RX_1: now also U4.20 (RXD), J2.3 (Pin_3); no longer U3.20 (RXD)
- net RX_2: now also U3.20 (RXD), J4.3 (Pin_3); no longer U4.20 (RXD)
- net RX_3: now also J5.3 (Pin_3)
- net TX_0: now also J1.2 (Pin_2)
- net TX_1: now also U4.21 (TXD), J2.2 (Pin_2); no longer U3.21 (TXD)
- net TX_2: now also U3.21 (TXD), J4.2 (Pin_2); no longer U4.21 (TXD)
- net TX_3: now also J5.2 (Pin_2)
- net U1_OUT+: now also U4.3 (D+); no longer U3.3 (D+)
- net U1_OUT-: now also U4.4 (D-); no longer U3.4 (D-)
- net U2_OUT+: now also U3.3 (D+); no longer U4.3 (D+)
- net U2_OUT-: now also U3.4 (D-); no longer U4.4 (D-)
- net VBUS: now also C17.1, C19.1, C20.1, C22.1, JP1.1 (A), JP2.1 (A), JP3.1 (A), JP4.1 (A), U5.3 (VI); no longer U1.7 (REGIN), U3.7 (REGIN), U4.7 (REGIN), U6.7 (REGIN)
- net at U1.13 (GPIO.1): now also D4.1 (K)
- net at U1.14 (GPIO.0): now also D7.1 (K)
- net at U1.9 (~{RSTb}): now also R27.1
- net at U3.13 (GPIO.1): now also D3.1 (K)
- net at U3.14 (GPIO.0): now also D6.1 (K)
- net at U3.15 (~{SUSPENDb}): now also R29.2; no longer R22.2
- net at U3.9 (~{RSTb}): now also R26.1
- net at U4.15 (~{SUSPENDb}): now also R30.2; no longer R23.2
- net at U6.15 (~{SUSPENDb}): now also R33.2; no longer R24.2
- net at U6.13 (GPIO.1): now also D9.1 (K)
- net at U6.14 (GPIO.0): now also D10.1 (K)
- net at U6.9 (~{RSTb}): now also R32.1
- net at U4.13 (GPIO.1): now also D5.1 (K)
- net at U4.14 (GPIO.0): now also D8.1 (K)
- net at U4.9 (~{RSTb}): now also R28.1
- new net: D5.2 (A), D8.2 (A), R24.1
- new net: D4.2 (A), D7.2 (A), R23.1
- new net: J1.1 (Pin_1), JP1.2 (B)
- new net: J5.1 (Pin_1), JP4.2 (B)
- new net: J4.1 (Pin_1), JP3.2 (B)
- new net: D3.2 (A), D6.2 (A), R22.1
- new net: D10.2 (A), D9.2 (A), R31.1
- new net: J2.1 (Pin_1), JP2.2 (B)
- no-connect marks 55 -> 35
Other:
- moved on the sheet: C1, C10, C11, C12, C13, C18, C3, C4, C5, C6, C7, C8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
